File: nRF development board HAN_V1.0/MCU.kicad_sch (KiCad schematic)
At the start: 11 parts, among them J3 U.FL-R-SMT-1_10_, J4 Conn_02x05_Top_Bottom, U3 NRF5340-QKAA-R7, Y1 32mHz

Commit message: Updated schematic
Changed lines of the file:
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@@
     (effects (font (size 1.27 1.27)) (justify left bottom))
+  )
+  (hierarchical_label "GPS_PPS" (shape output) (at 378.46 73.66 180) (fields_autoplaced)
+    (effects (font (size 1.27 1.27)) (justify right))
   )
   (hierarchical_label "ERR" (shape output) (at 69.85 87.63 0) (fields_autoplaced)
@@
     (effects (font (size 1.27 1.27)) (justify left))
   )
+  (hierarchical_label "IMU_INT" (shape output) (at 378.46 113.03 180) (fields_autoplaced)
+    (effects (font (size 1.27 1.27)) (justify right))
+  )
   (hierarchical_label "USB_D-" (shape bidirectional) (at 93.98 269.24 180) (fields_autoplaced)
     (effects (font (size 1.27 1.27)) (justify right))
@@
     (effects (font (size 1.27 1.27)) (justify right))
   )
+  (hierarchical_label "MIC_SELECT" (shape input) (at 378.46 92.71 180) (fields_autoplaced)
+    (effects (font (size 1.27 1.27)) (justify right))
+  )
   (hierarchical_label "UART_TX" (shape input) (at 71.12 139.7 0) (fields_autoplaced)
     (effects (font (size 1.27 1.27)) (justify left))
@@
   (hierarchical_label "CHG" (shape output) (at 69.85 90.17 0) (fields_autoplaced)
     (effects (font (size 1.27 1.27)) (justify left))
+  )
+  (hierarchical_label "ENC_SW" (shape output) (at 378.46 132.08 180) (fields_autoplaced)
+    (effects (font (size 1.27 1.27)) (justify right))
+  )
+  (hierarchical_label "ENC_A" (shape output) (at 378.46 129.54 180) (fields_autoplaced)
+    (effects (font (size 1.27 1.27)) (justify right))
+  )
+  (hierarchical_label "SW1" (shape output) (at 378.46 86.36 180) (fields_autoplaced)
+    (effects (font (size 1.27 1.27)) (justify right))
   )
   (hierarchical_label "BAT_MON" (shape output) (at 69.85 105.41 0) (fields_autoplaced)
@@
     (effects (font (size 1.27 1.27)) (justify left))
   )
+  (hierarchical_label "SW2" (shape output) (at 378.46 83.82 180) (fields_autoplaced)
+    (effects (font (size 1.27 1.27)) (justify right))
+  )
+  (hierarchical_label "GES_INT" (shape output) (at 377.19 121.92 180) (fields_autoplaced)
+    (effects (font (size 1.27 1.27)) (justify right))
+  )
+  (hierarchical_label "MIC_WS" (shape output) (at 378.46 95.25 180) (fields_autoplaced)
+    (effects (font (size 1.27 1.27)) (justify right))
+  )
   (hierarchical_label "SPI_CLK" (shape input) (at 71.12 119.38 0) (fields_autoplaced)
     (effects (font (size 1.27 1.27)) (justify left))
+  )
+  (hierarchical_label "MIC_BCLK" (shape output) (at 378.46 97.79 180) (fields_autoplaced)
+    (effects (font (size 1.27 1.27)) (justify right))
   )
   (hierarchical_label "SPI_CS" (shape input) (at 71.12 121.92 0) (fields_autoplaced)
     (effects (font (size 1.27 1.27)) (justify left))
   )
+  (hierarchical_label "IMU_PS1" (shape input) (at 378.46 107.95 180) (fields_autoplaced)
+    (effects (font (size 1.27 1.27)) (justify right))
+  )
+  (hierarchical_label "IMU_PS0" (shape input) (at 378.46 105.41 180) (fields_autoplaced)
+    (effects (font (size 1.27 1.27)) (justify right))
+  )
   (hierarchical_label "LOW_BAT" (shape input) (at 69.85 100.33 0) (fields_autoplaced)
     (effects (font (size 1.27 1.27)) (justify left))
+  )
+  (hierarchical_label "ENC_B" (shape output) (at 378.46 134.62 180) (fields_autoplaced)
+    (effects (font (size 1.27 1.27)) (justify right))
+  )
+  (hierarchical_label "MIC_DATA" (shape output) (at 378.46 100.33 180) (fields_autoplaced)
+    (effects (font (size 1.27 1.27)) (justify right))
   )
   (hierarchical_label "I2C_SDA" (shape input) (at 71.12 132.08 0) (fields_autoplaced)
@@
     (effects (font (size 1.27 1.27)) (justify left))
   )
+  (hierarchical_label "~{IMU_RST}" (shape input) (at 378.46 110.49 180) (fields_autoplaced)
+    (effects (font (size 1.27 1.27)) (justify right))
+  )
   (hierarchical_label "SHPACT" (shape input) (at 69.85 92.71 0) (fields_autoplaced)
     (effects (font (size 1.27 1.27)) (justify left))
   )
+  (hierarchical_label "SW3" (shape output) (at 378.46 81.28 180) (fields_autoplaced)
+    (effects (font (size 1.27 1.27)) (justify right))
+  )
   (netclass_flag "" (length 2.54) (shape round) (at 68.58 240.03 0) (fields_autoplaced)

Commit message: QOL update
Parts:
- renumbered C13 to C33, C13 to C34, C13 to C35, L1 to L6
