File: nRF development board HAN_V1.0/USB.kicad_sch (KiCad schematic)
At the start: 13 parts, among them J2 USB_C_Receptacle_USB2.0

Commit message: QOL update
Parts:
- renumbered R5 to R13, R5 to R14, R5 to R15
