File: nRF development board HAN_V1.0/Power.kicad_sch (KiCad schematic)
At the start: 55 parts, among them J1 Conn_01x03_Pin, Q1 DMC2400UV, Q2 FDV303N, SW1 SW_Push, U1 NPM1100-QDAA-R, U1 NRF5340-QKAA-R7, U2 XC9236F08CER-G

Commit message: QOL update
Parts:
- renumbered U1 to U3

Commit message: Updated PCB
Other:
- moved on the sheet: C24, C25, C26, C27
