File: nRF development board HAN_V1.0/nRF development board HAN_V1.0.kicad_pcb (KiCad board)
At the start: 4 copper layers, 78 parts, among them J1 Conn_01x03_Pin, J2 USB_C_Receptacle_USB2.0, J3 U.FL-R-SMT-1_10_, J4 Conn_02x05_Top_Bottom, Q1 DMC2400UV, Q2 FDV303N, SW1 SW_Push, U1 NPM1100-QDAA-R, U2 XC9236F08CER-G, U3 NRF5340-QKAA-R7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

Commit message: Backups
Parts:
- added MK1: SPH0645LM4H, Sensor_Audio:Knowles_SPH0645LM4H-6_3.5x2.65mm, F.Cu at (163.4, 112.1)
- added SW3: SW_Push, Button_Switch_SMD:SW_SPST_PTS810, F.Cu at (157.7, 106.2)
- added SW4: SW_Push, Button_Switch_SMD:SW_SPST_PTS810, F.Cu at (157.7, 111.0)
- added SW5: SW_Push, Button_Switch_SMD:SW_SPST_PTS810, F.Cu at (157.7, 115.7)
- added U4: BME280, Package_LGA:Bosch_LGA-8_2.5x2.5mm_P0.65mm_ClockwisePinNumbering, F.Cu at (163.0, 116.7)
- added U5: BNO055, Package_LGA:LGA-28_5.2x3.8mm_P0.5mm, F.Cu at (164.6, 106.6)

Commit message: Updated PCB
Parts:
- added C36: 100nF, Capacitor_SMD:C_0603_1608Metric_Pad1.08x0.95mm_HandSolder, F.Cu at (42.5, 136.6)
- added C37: 1.0uF, Capacitor_SMD:C_0603_1608Metric_Pad1.08x0.95mm_HandSolder, F.Cu at (42.5, 139.1)
- added C38: 100nF, Capacitor_SMD:C_0603_1608Metric_Pad1.08x0.95mm_HandSolder, F.Cu at (42.5, 141.6)
- added C39: 100nF, Capacitor_SMD:C_0603_1608Metric_Pad1.08x0.95mm_HandSolder, F.Cu at (42.5, 144.2)
- added C40: 22pF, Capacitor_SMD:C_0603_1608Metric_Pad1.08x0.95mm_HandSolder, F.Cu at (42.5, 146.7)
- added C41: 22pF, Capacitor_SMD:C_0603_1608Metric_Pad1.08x0.95mm_HandSolder, F.Cu at (42.5, 149.2)
- added C42: 100nF, Capacitor_SMD:C_0603_1608Metric_Pad1.08x0.95mm_HandSolder, F.Cu at (46.9, 136.6)
- added C43: 1.0uF, Capacitor_SMD:C_0603_1608Metric_Pad1.08x0.95mm_HandSolder, F.Cu at (46.9, 139.1)
- added C44: 220pF, Capacitor_SMD:C_0603_1608Metric_Pad1.08x0.95mm_HandSolder, F.Cu at (46.9, 141.6)
- added C45: 1.0uF, Capacitor_SMD:C_0603_1608Metric_Pad1.08x0.95mm_HandSolder, F.Cu at (46.9, 144.2)
- added C46: 100nF, Capacitor_SMD:C_0603_1608Metric_Pad1.08x0.95mm_HandSolder, F.Cu at (46.9, 146.7)
- added C47: 100nF, Capacitor_SMD:C_0603_1608Metric_Pad1.08x0.95mm_HandSolder, F.Cu at (46.9, 149.2)
- added C48: 100nF, Capacitor_SMD:C_0603_1608Metric_Pad1.08x0.95mm_HandSolder, F.Cu at (51.2, 136.6)
- added C49: 100nF, Capacitor_SMD:C_0603_1608Metric_Pad1.08x0.95mm_HandSolder, F.Cu at (51.2, 139.1)
- added C50: 100nF, Capacitor_SMD:C_0603_1608Metric_Pad1.08x0.95mm_HandSolder, F.Cu at (51.2, 141.6)
- added C51: 100nF, Capacitor_SMD:C_0603_1608Metric_Pad1.08x0.95mm_HandSolder, F.Cu at (51.2, 144.2)
- added C52: 100nF, Capacitor_SMD:C_0603_1608Metric_Pad1.08x0.95mm_HandSolder, F.Cu at (51.2, 146.7)
- added D6: CUS520,H3F, SamacSys:SOD2513X115N, F.Cu at (55.9, 146.5)
- added U6: TSL25911FN, SamacSys:TSL25911FN, F.Cu at (56.3, 138.1)
- added U7: FGPMMOPA6H, SamacSys:FGPMMOPA6H, F.Cu at (58.9, 118.9)
- added U8: APDS-9960, Sensor:Avago_APDS-9960, F.Cu at (56.4, 142.8)
- D1: footprint SamacSys_Parts:MBRM110LT1G -> SamacSys:MBRM110LT1G
- Q1: footprint SamacSys_Parts:SOTFL50P162X60-6N -> SamacSys:SOTFL50P162X60-6N
- Q2: footprint SamacSys_Parts:SOT96P237X111-3N -> SamacSys:SOT96P237X111-3N
- U1: footprint SamacSys_Parts:QFN50P400X400X90-25N-D -> SamacSys:QFN50P400X400X90-25N-D
- U2: footprint SamacSys_Parts:XC9236F08CERG -> SamacSys:XC9236F08CERG
Connections:
- MK1 pad 1: unconnected-(MK1-WS-Pad1) -> /MCU/MIC_WS
- MK1 pad 2: unconnected-(MK1-SEL-Pad2) -> /MCU/MIC_SELECT
- MK1 pad 3: unconnected-(MK1-GND-Pad3) -> GNDD
- MK1 pad 4: unconnected-(MK1-BCLK-Pad4) -> /MCU/MIC_BCLK
- MK1 pad 5: unconnected-(MK1-VDD-Pad5) -> +3V3
- MK1 pad 6: unconnected-(MK1-DATA-Pad6) -> Net-(MK1-DATA)
- SW3 pad 1: unconnected-(SW3-Pad1) -> /MCU/SW1
- SW3 pad 2: unconnected-(SW3-Pad2) -> GNDD
- SW4 pad 1: unconnected-(SW4-Pad1) -> /MCU/SW2
- SW4 pad 2: unconnected-(SW4-Pad2) -> GNDD
- SW5 pad 1: unconnected-(SW5-Pad1) -> /MCU/SW3
- SW5 pad 2: unconnected-(SW5-Pad2) -> GNDD
- U4 pad 1: unconnected-(U4-GND-Pad1) -> GNDD
- U4 pad 2: unconnected-(U4-CSB-Pad2) -> /Actuators/SPI_CS
- U4 pad 3: unconnected-(U4-SDI-Pad3) -> /Actuators/SPI_MOSI
- U4 pad 4: unconnected-(U4-SCK-Pad4) -> /Actuators/SPI_CLK
- U4 pad 5: unconnected-(U4-SDO-Pad5) -> /Actuators/SPI_MISO
- U4 pad 6: unconnected-(U4-VDDIO-Pad6) -> +3V3
- U4 pad 7: unconnected-(U4-GND-Pad7) -> GNDD
- U4 pad 8: unconnected-(U4-VDD-Pad8) -> +3V3
- U5 pad 10: unconnected-(U5-BL_IND-Pad10) -> GNDD
- U5 pad 11: unconnected-(U5-~{RESET}-Pad11) -> /MCU/~{IMU_RST}
- U5 pad 14: unconnected-(U5-INT-Pad14) -> /MCU/IMU_INT
- U5 pad 15: Net-(U5-GNDIO-Pad15) -> GNDD
- U5 pad 16: Net-(U5-GNDIO-Pad15) -> GNDD
- U5 pad 17: unconnected-(U5-COM3-Pad17) -> Net-(U5-COM3)
- U5 pad 18: unconnected-(U5-COM2-Pad18) -> GNDD
- U5 pad 19: unconnected-(U5-COM1-Pad19) -> /Actuators/I2C_SCL
- U5 pad 2: unconnected-(U5-GND-Pad2) -> GNDD
- U5 pad 20: unconnected-(U5-COM0-Pad20) -> /Actuators/I2C_SDA
- U5 pad 25: Net-(U5-GNDIO-Pad15) -> GNDD
- U5 pad 26: unconnected-(U5-XOUT32-Pad26) -> Net-(U5-XOUT32)
- U5 pad 27: unconnected-(U5-XIN32-Pad27) -> Net-(U5-XIN32)
- U5 pad 28: unconnected-(U5-VDDIO-Pad28) -> +3V3
- U5 pad 3: unconnected-(U5-VDD-Pad3) -> +3V3
- U5 pad 4: unconnected-(U5-~{BOOT_LOAD_PIN}-Pad4) -> +3V3
- U5 pad 5: unconnected-(U5-PS1-Pad5) -> /MCU/IMU_PS1
- U5 pad 6: unconnected-(U5-PS0-Pad6) -> /MCU/IMU_PS0
- U5 pad 9: unconnected-(U5-CAP-Pad9) -> Net-(U5-CAP)
