File: nRF development board HAN_V1.0/nRF development board HAN_V1.0.kicad_sch (KiCad schematic)
At the start: 0 parts

Commit message: Updated schematic
Other:
- sheet Actuators ports: added none; removed UART_RX, UART_TX
- sheet MCU ports: added ENC_A, ENC_B, ENC_SW, GES_INT, GPS_PPS, IMU_INT, IMU_PS0, IMU_PS1, MIC_BCLK, MIC_DATA, MIC_SELECT, MIC_WS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; removed none
- sheet Sensors ports: added ENC_A, ENC_B, ENC_SW, GES_INT, GPS_PPS, GPS_RX, GPS_TX, IMU_INT, IMU_PS0, IMU_PS1, MIC_BCLK, MIC_DATA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; removed UART_RX, UART_TX
